File: pcb/storybox.kicad_sch (KiCad schematic)
At the start: 26 parts, among them J1 Conn_01x01_Pin, J3 Speaker, J4 Ext, J5 AudioJack, SW1 Prev, SW2 Next, SW3 Play, SW4 Home, U1 Pico, U2 Amplifier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

Commit message: dernière version de la pcb + schéma
Parts:
- Battery1: symbol Connector:Jack-DC -> storybox:polarized_connector
- J3: symbol Connector:Screw_Terminal_01x02 -> storybox:polarized_connector
Changed lines of the file:
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@@
+	(wire
+		(pts
+			(xy 212.09 71.12) (xy 212.09 77.47)
+		)
+		(stroke
+			(width 0)
+			(type default)
+		)
+	)
 	(wire
 		(pts
@@
 	(wire
 		(pts
+			(xy 105.41 38.1) (xy 105.41 52.07)
+		)
+		(stroke
+			(width 0)
+			(type default)
+		)
+	)
+	(wire
+		(pts
 			(xy 181.61 156.21) (xy 175.26 156.21)
 		)
@@
 	(wire
 		(pts
+			(xy 100.33 41.91) (xy 102.87 41.91)
+		)
+		(stroke
+			(width 0)
+			(type default)
+		)
+	)
+	(wire
+		(pts
 			(xy 83.82 106.68) (xy 83.82 107.95)
 		)
@@
 	(wire
 		(pts
+			(xy 209.55 71.12) (xy 209.55 80.01)
+		)
+		(stroke
+			(width 0)
+			(type default)
+		)
+	)
+	(wire
+		(pts
 			(xy 133.35 90.17) (xy 119.38 90.17)
 		)
@@
 	(wire
 		(pts
-			(xy 105.41 50.8) (xy 105.41 38.1)
-		)
-		(stroke
-			(width 0)
-			(type default)
-		)
-	)
-	(wire
-		(pts
 			(xy 132.08 73.66) (xy 138.43 73.66)
 		)
@@
 	(wire
 		(pts
+			(xy 102.87 41.91) (xy 102.87 52.07)
+		)
+		(stroke
+			(width 0)
+			(type default)
+		)
+	)
+	(wire
+		(pts
 			(xy 181.61 171.45) (xy 160.02 171.45)
 		)
@@
 	(wire
 		(pts
-			(xy 209.55 74.93) (xy 209.55 80.01)
-		)
-		(stroke
-			(width 0)
-			(type default)
-		)
-	)
-	(wire
-		(pts
-			(xy 100.33 41.91) (xy 100.33 50.8)
-		)
-		(stroke
-			(width 0)
-			(type default)
-		)
-	)
-	(wire
-		(pts
 			(xy 147.32 71.12) (xy 147.32 72.39)
 		)
@@
 	(wire
 		(pts
-			(xy 212.09 77.47) (xy 212.09 74.93)
-		)
-		(stroke
-			(width 0)
-			(type default)
-		)
-	)
-	(wire
-		(pts
 			(xy 26.67 127) (xy 26.67 144.78)
 		)
@@
 	)
 	(symbol
-		(lib_id "Connector:Jack-DC")
-		(at 102.87 58.42 270)
-		(mirror x)
+		(lib_id "storybox:polarized_connector")
+		(at 107.95 52.07 270)
 		(unit 1)
 		(exclude_from_sim no)
@@
 		(dnp no)
 		(property "Reference" "Battery1"
-			(at 97.79 57.1499 90)
+			(at 99.314 55.626 90)
 			(effects
 				(font
@@
 		)
 		(property "Value" "4.2V"
-			(at 97.79 59.6899 90)
+			(at 99.314 58.166 90)
 			(effects
 				(font
@@
 		)
 		(property "Footprint" "storybox:connector_polarized"
-			(at 101.854 57.15 0)
+			(at 107.95 52.07 0)
 			(effects
 				(font
@@
 		)
 		(property "Datasheet" "~"
-			(at 101.854 57.15 0)
+			(at 107.95 52.07 0)
 			(effects
 				(font
@@
 		)
 		(property "Description" "DC Barrel Jack"
-			(at 102.87 58.42 0)
+			(at 107.95 52.07 0)
 			(effects
 				(font
@@
 	)
 	(symbol
-		(lib_id "Connector:Screw_Terminal_01x02")
-		(at 212.09 69.85 270)
+		(lib_id "storybox:polarized_connector")
+		(at 214.63 71.12 270)
 		(mirror x)
 		(unit 1)
@@
 		(dnp no)
 		(property "Reference" "J3"
-			(at 212.0901 67.31 0)
+			(at 211.074 61.468 0)
 			(effects
 				(font
@@
 		)
 		(property "Value" "Speaker"
-			(at 209.5501 67.31 0)
+			(at 215.9 67.564 0)
 			(effects
 				(font
@@
 		)
 		(property "Footprint" "storybox:connector_polarized"
-			(at 212.09 69.85 0)
+			(at 214.63 71.12 0)
 			(effects
 				(font
@@
 		)
 		(property "Datasheet" "~"
-			(at 212.09 69.85 0)
+			(at 214.63 71.12 0)
 			(effects
 				(font
@@
 		)
 		(property "Description" "Generic screw terminal, single row, 01x02, script generated (kicad-library-utils/schlib/autogen/connector/)"
-			(at 212.09 69.85 0)
-			(effects
-				(font
+			(at 214.63 71.12 0)
+			(effects
+				(font
